File: MRCS-Nano-Grade-Xing-Breakout.brd (EAGLE design)
At the start: 99.8 x 68.8 mm, 20 parts, among them CON1 5V PWR, J1 5V PWR, J2 Unused I/O, J4 Outputs

Commit message: gerb files for first build
Parts:
- added U$3: (no value), MRCSLogoTop:MRCSLOGOTOP
Other:
- board text added: "5VDC"
- board text added: "Grade Xing Breakout"
- board text removed: "5DVC"
- board text removed: "Grade XING Breakout"
Changed lines of the file:
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@@
 <text x="91.44" y="58.42" size="1.4224" layer="51" font="vector" rot="R180">V1.0 20220314</text>
 <text x="34.29" y="40.64" size="1.778" layer="51" font="vector">Arduino Nano</text>
-<text x="91.44" y="62.23" size="1.4224" layer="51" font="vector" rot="R180">Grade XING Breakout</text>
+<text x="91.44" y="62.23" size="1.4224" layer="51" font="vector" rot="R180">Grade Xing Breakout</text>
 <text x="43.18" y="60.96" size="2.794" layer="51" font="vector" ratio="10">+GBG+L+L
 5NLN5152</text>
@@
 <text x="33.655" y="1.27" size="2.794" layer="52" font="vector" ratio="10">4+5+6+7+</text>
 <text x="59.055" y="3.81" size="3.81" layer="51" font="vector" ratio="10">5G5G</text>
-<text x="76.835" y="3.81" size="3.81" layer="51" font="vector" ratio="10">5DVC</text>
+<text x="76.835" y="3.81" size="3.81" layer="51" font="vector" ratio="10">5VDC</text>
 <text x="10.16" y="1.27" size="2.794" layer="51" font="vector" ratio="10">05152535</text>
 <text x="33.02" y="1.27" size="2.794" layer="51" font="vector" ratio="10">45556575</text>
@@
 <element name="U$2" library="MRCS-prop65warningBtm" package="CA-PROP65WARNING" value="" x="46.99" y="50.8"/>
 <element name="J2" library="SPCoast" package="1X08_LOCK" value="Unused I/O" x="5.08" y="43.18" rot="R270"/>
+<element name="U$3" library="MRCSLogoTop" package="MRCSLOGOTOP" value="" x="69.85" y="45.72"/>
 </elements>
 <signals>
@@
 </signal>
 </signals>
+<errors>
+</errors>
 </board>
 </drawing>
